Commit message: add base_footprint link

File: mirte_description/mirte_master_description/urdf/mirte_master.xacro (robot description, xacro)
@@ -162,4 +162,11 @@
     </joint>
   </xacro:if>
+  <xacro:property name="wheel_zoff" value="0.05"/>
+   <link name="base_footprint"/>
+   <joint name="base_joint" type="fixed">
+     <parent link="base_link"/>
+     <child link="base_footprint"/>
+     <origin xyz="0.0 0.0 ${-(wheel_radius + wheel_zoff)}" rpy="0 0 0"/>
+   </joint>
   <xacro:if value="$(arg sonar_enable)">
     <xacro:include filename="$(find mirte_master_description)/urdf/ultrasonic.xacro" />
